Commit message: Fixed gazebo and rviz simulation alignment and script to run bow motion.  Gazebo's center of gravity is still an issue though.

File: bioloid_description/urdf/part2_typea.urdf (robot description, URDF)
Before this commit: robot typea, 28 links, 27 joints
Links:
- link base_link: mass 1.0 -> 0.25
Joints:
- joint l_ankle_lateral_joint: axis 0 0 1 -> 0 0 -1
- joint l_ankle_swing_joint: limit lower=-2.0 upper=2.0 effort=10 velocity=5.6548668 -> lower=-2.0 upper=0.4 effort=10 velocity=5.6548668
- joint l_hip_lateral_joint: axis 0 0 1 -> 0 0 -1
- joint l_knee_joint: axis 0 0 1 -> 0 0 -1
- joint r_ankle_lateral_joint: axis 0 0 1 -> 0 0 -1
- joint r_ankle_swing_joint: limit lower=-2.0 upper=2.0 effort=10 velocity=5.6548668 -> lower=-0.4 upper=2.0 effort=10 velocity=5.6548668
- joint r_elbow_joint: axis 0 0 1 -> 0 0 -1
- joint r_hip_lateral_joint: axis 0 0 1 -> 0 0 -1
- joint r_knee_joint: axis 0 0 1 -> 0 0 -1; limit lower=0 upper=2 effort=10 velocity=5.6548668 -> lower=-2 upper=0 effort=10 velocity=5.6548668
- joint r_shoulder_lateral_joint: axis 0 0 1 -> 0 0 -1

File: bioloid_description/urdf/typea.urdf (robot description, URDF)
Before this commit: robot typea, 27 links, 26 joints
Joints:
- joint head2_joint: type revolute -> fixed
- joint l_ankle_swing_joint: limit lower=-2.0 upper=0.3999999999999999 effort=10 velocity=5.6548668 -> lower=-2.0 upper=0.4 effort=10 velocity=5.6548668
- joint l_hip_swing_joint: limit lower=-0.3999999999999999 upper=2.0 effort=10 velocity=5.6548668 -> lower=-2.0 upper=2.0 effort=10 velocity=5.6548668
- joint r_ankle_swing_joint: limit lower=-0.3999999999999999 upper=2.0 effort=10 velocity=5.6548668 -> lower=-0.4 upper=2.0 effort=10 velocity=5.6548668
- joint r_elbow_joint: axis 0 0 1 -> 0 0 -1
- joint r_hip_swing_joint: limit lower=-2.0 upper=0.3999999999999999 effort=10 velocity=5.6548668 -> lower=-2.0 upper=2.0 effort=10 velocity=5.6548668
- joint r_knee_joint: limit lower=-2 upper=00000 effort=10 velocity=5.6548668 -> lower=-2 upper=0 effort=10 velocity=5.6548668
- joint r_shoulder_lateral_joint: axis 0 0 1 -> 0 0 -1

Commit message: Fixed the initial pos of hip_twist_joint to match with real robot.

File: bioloid_description/urdf/part2_typea.urdf (robot description, URDF)
Before this commit: robot typea, 28 links, 27 joints
Joints:
- joint l_hip_twist_joint: limit lower=-0.5 upper=0.5 effort=10 velocity=5.6548668 -> lower=-0.8 upper=0.8 effort=10 velocity=5.6548668; origin xyz=0 0.0385 -0.0655 rpy=0 3.141592653589793 -1.5707963267948966 -> xyz=0 0.0385 -0.0655 rpy=0 3.141592653589793 -0.788
- joint r_hip_twist_joint: limit lower=-0.5 upper=0.5 effort=10 velocity=5.6548668 -> lower=-0.8 upper=0.8 effort=10 velocity=5.6548668; origin xyz=0 -0.0385 -0.0655 rpy=0 3.141592653589793 1.5707963267948966 -> xyz=0 -0.0385 -0.0655 rpy=0 3.141592653589793 0.788

File: bioloid_description/urdf/typea.urdf (robot description, URDF)
Before this commit: robot typea, 27 links, 26 joints
Joints:
- joint l_hip_twist_joint: limit lower=-0.5 upper=0.5 effort=10 velocity=5.6548668 -> lower=-0.8 upper=0.8 effort=10 velocity=5.6548668; origin xyz=0 0.0385 -0.0655 rpy=0 3.141592653589793 -1.5707963267948966 -> xyz=0 0.0385 -0.0655 rpy=0 3.141592653589793 -0.788
- joint r_hip_twist_joint: limit lower=-0.5 upper=0.5 effort=10 velocity=5.6548668 -> lower=-0.8 upper=0.8 effort=10 velocity=5.6548668; origin xyz=0 -0.0385 -0.0655 rpy=0 3.141592653589793 1.5707963267948966 -> xyz=0 -0.0385 -0.0655 rpy=0 3.141592653589793 0.788

Commit message: Created tasks motion files.

File: bioloid_description/urdf/part2_typea.urdf (robot description, URDF)
Before this commit: robot typea, 28 links, 27 joints
Links:
- removed link world
- link torso_link: mass 3.4770266466 -> 1.5
Joints:
- removed joint fixed_base

Commit message: Modifieed the script to take motion files more flexibly.

File: bioloid_description/urdf/part2_typea.urdf (robot description, URDF)
Before this commit: robot typea, 27 links, 26 joints
Links:
- added link world
- link torso_link: mass 1.5 -> 0.25
Joints:
- added joint fixed_base: type fixed, parent world, child base_link, origin xyz=0 0 0 rpy=0 0 0
- joint l_hip_twist_joint: origin xyz=0 0.0385 -0.0655 rpy=0 3.141592653589793 -0.788 -> xyz=0 0.0385 -0.0655 rpy=0 3.141592653589793 -1.5707963267948966

Commit message: Fixed .stl orientation with new ones from Aspose.

File: bioloid_description/urdf/part2_typea.urdf (robot description, URDF)
Before this commit: robot typea, 28 links, 27 joints
Joints:
- joint head2_joint: origin xyz=0 0 0 rpy=-1.57 0 0 -> xyz=0 0 0 rpy=0 0 0
- joint head_joint: origin xyz=0 0 0 rpy=-1.57 0 0 -> xyz=0 0 0 rpy=0 0 0

Commit message: Fixed Gazebo camera pose to use ~/.gz/sim/8/gui.config.  But no gravity still causes robot float up.

File: bioloid_description/urdf/part2_typea.urdf (robot description, URDF)
Before this commit: robot typea, 28 links, 27 joints
Links:
- removed link world
Joints:
- removed joint fixed_base
- joint l_hip_twist_joint: origin xyz=0 0.0385 -0.0655 rpy=0 3.141592653589793 -1.5707963267948966 -> xyz=0 0.0385 -0.0655 rpy=0 3.141592653589793 -0.788

Commit message: Cleaned up and tried more gravity controls but not so successful still.

File: bioloid_description/urdf/part2_typea.urdf (robot description, URDF)
Before this commit: robot typea, 27 links, 26 joints
Links:
- link base_link: mass 0.25 -> None
