Commit message: Fixed joint alignment and real robot joint control.

File: bioloid_description/urdf/typea.urdf (robot description, URDF)
Before this commit: robot typea, 27 links, 26 joints
Joints:
- joint l_ankle_lateral_joint: axis 0 0 1 -> 0 0 -1
- joint l_hip_lateral_joint: axis 0 0 1 -> 0 0 -1
- joint l_knee_joint: axis 0 0 1 -> 0 0 -1; limit lower=-2 upper=0 effort=10 velocity=5.6548668 -> lower=0 upper=2 effort=10 velocity=5.6548668
- joint r_ankle_lateral_joint: axis 0 0 1 -> 0 0 -1
- joint r_hip_lateral_joint: axis 0 0 1 -> 0 0 -1
- joint r_knee_joint: axis 0 0 1 -> 0 0 -1; limit lower=0 upper=2 effort=10 velocity=5.6548668 -> lower=-2 upper=00000 effort=10 velocity=5.6548668

Commit message: Cleened up.  Tested IMU sim but failed to balance still.

File: bioloid_description/urdf/typea.urdf (robot description, URDF)
Before this commit: robot typea, 27 links, 26 joints
Links:
- link head2_link: mass 0.1 -> None
- link head_link: mass 0.1 -> None
- link imu_link: mass 0.001 -> None
- link l_ankle_lateral_link: mass 0.1867801099 -> None
- link l_ankle_swing_link: mass 0.6852429363 -> None
- link l_foot_link: mass 0.1867801099 -> None
- link l_hand_link: mass 0.0303003163 -> None
- link l_hip_lateral_link: mass 0.6852429363 -> None
- link l_hip_twist_link: mass 0.0755193623 -> None
- link l_lower_arm_link: mass 0.3822870734 -> None
- link l_lower_leg_link: mass 0.4326089335 -> None
- link l_shoulder_swing_link: mass 0.0595945816 -> None
- link l_upper_arm_link: mass 0.3822870734 -> None
- link l_upper_leg_link: mass 0.1557654222 -> None
- link r_ankle_lateral_link: mass 0.1867801099 -> None
- link r_ankle_swing_link: mass 0.6852429363 -> None
- link r_foot_link: mass 0.1867801099 -> None
- link r_hand_link: mass 0.0303003163 -> None
- link r_hip_lateral_link: mass 0.6852429363 -> None
- link r_hip_twist_link: mass 0.0755193623 -> None
- link r_lower_arm_link: mass 0.3833833954 -> None
- link r_lower_leg_link: mass 0.4326089335 -> None
- link r_shoulder_swing_link: mass 0.0595945816 -> None
- link r_upper_arm_link: mass 0.3822870734 -> None
- link r_upper_leg_link: mass 0.1557654222 -> None
- link torso_link: mass 3.4770266466 -> None

File: bioloid_description/urdf/typea_gz_ros2ctl.urdf (robot description, URDF)
Before this commit: robot typea, 27 links, 26 joints
Links:
- link imu_link: mass 0.001 -> None
- link torso_link: mass 0.25 -> None

Commit message: Changing the inertia and CoM of each link but not yet finished...

File: bioloid_description/urdf/typea.urdf (robot description, URDF)
Before this commit: robot typea, 27 links, 26 joints
Links:
- link head2_link: mass None -> 0.06; geometry collision box size=0.04 0.10 0.08; visual mesh filename=package://bioloid_description/assets/cad/Bioloid_CUERPO_vis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
- link head_link: mass None -> 0.05
- link l_ankle_lateral_link: mass None -> 0.015
- link l_ankle_swing_link: mass None -> 0.0685
- link l_foot_link: mass None -> 0.015
- link l_hand_link: mass None -> 0.008
- link l_hip_lateral_link: mass None -> 0.120
- link l_hip_twist_link: mass None -> 0.016
- link l_lower_arm_link: mass None -> 0.060
- link l_lower_leg_link: mass None -> 0.080
- link l_shoulder_swing_link: mass None -> 0.010
- link l_upper_arm_link: mass None -> 0.070
- link l_upper_leg_link: mass None -> 0.030
- link r_ankle_lateral_link: mass None -> 0.015
- link r_ankle_swing_link: mass None -> 0.0685
- link r_foot_link: mass None -> 0.015
- link r_hand_link: mass None -> 0.008
- link r_hip_lateral_link: mass None -> 0.120
- link r_hip_twist_link: mass None -> 0.016
- link r_lower_arm_link: mass None -> 0.060
- link r_lower_leg_link: mass None -> 0.080
- link r_shoulder_swing_link: mass None -> 0.010
- link r_upper_arm_link: mass None -> 0.070
- link r_upper_leg_link: mass None -> 0.030
- link torso_link: mass None -> 0.411
