Commit message: Cleaned up the other 2 URDF files.

File: bioloid_description/urdf/typea_cmdpos.urdf (robot description, URDF)
Before this commit: robot typea, 27 links, 26 joints
Links:
- link head2_link: mass 0.1 -> 0.06; geometry collision box size=0.04 0.10 0.08; visual mesh filename=package://bioloid_description/assets/cad/Bioloid_CUERPO_vis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
- link head_link: mass 0.1 -> 0.05
- link imu_link: mass 0.001 -> None
- link l_ankle_lateral_link: mass 0.1867801099 -> 0.015
- link l_ankle_swing_link: mass 0.6852429363 -> 0.0685
- link l_foot_link: mass 0.1867801099 -> 0.015
- link l_hand_link: mass 0.0303003163 -> 0.008
- link l_hip_lateral_link: mass 0.6852429363 -> 0.120
- link l_hip_twist_link: mass 0.0755193623 -> 0.016
- link l_lower_arm_link: mass 0.3822870734 -> 0.060
- link l_lower_leg_link: mass 0.4326089335 -> 0.080
- link l_shoulder_swing_link: mass 0.0595945816 -> 0.010
- link l_upper_arm_link: mass 0.3822870734 -> 0.070
- link l_upper_leg_link: mass 0.1557654222 -> 0.030
- link r_ankle_lateral_link: mass 0.1867801099 -> 0.015
- link r_ankle_swing_link: mass 0.6852429363 -> 0.0685
- link r_foot_link: mass 0.1867801099 -> 0.015
- link r_hand_link: mass 0.0303003163 -> 0.008
- link r_hip_lateral_link: mass 0.6852429363 -> 0.120
- link r_hip_twist_link: mass 0.0755193623 -> 0.016
- link r_lower_arm_link: mass 0.3833833954 -> 0.060
- link r_lower_leg_link: mass 0.4326089335 -> 0.080
- link r_shoulder_swing_link: mass 0.0595945816 -> 0.010
- link r_upper_arm_link: mass 0.3822870734 -> 0.070
- link r_upper_leg_link: mass 0.1557654222 -> 0.030
- link torso_link: mass 0.25 -> 0.411

File: bioloid_description/urdf/typea_gz_ros2ctl.urdf (robot description, URDF)
Before this commit: robot typea, 27 links, 26 joints
Links:
- link head2_link: mass 0.1 -> 0.06; geometry collision box size=0.04 0.10 0.08; visual mesh filename=package://bioloid_description/assets/cad/Bioloid_CUERPO_vis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
- link head_link: mass 0.1 -> 0.05
- link l_ankle_lateral_link: mass 0.1867801099 -> 0.015
- link l_ankle_swing_link: mass 0.6852429363 -> 0.0685
- link l_foot_link: mass 0.1867801099 -> 0.015
- link l_hand_link: mass 0.0303003163 -> 0.008
- link l_hip_lateral_link: mass 0.6852429363 -> 0.120
- link l_hip_twist_link: mass 0.0755193623 -> 0.016
- link l_lower_arm_link: mass 0.3822870734 -> 0.060
- link l_lower_leg_link: mass 0.4326089335 -> 0.080
- link l_shoulder_swing_link: mass 0.0595945816 -> 0.010
- link l_upper_arm_link: mass 0.3822870734 -> 0.070
- link l_upper_leg_link: mass 0.1557654222 -> 0.030
- link r_ankle_lateral_link: mass 0.1867801099 -> 0.015
- link r_ankle_swing_link: mass 0.6852429363 -> 0.0685
- link r_foot_link: mass 0.1867801099 -> 0.015
- link r_hand_link: mass 0.0303003163 -> 0.008
- link r_hip_lateral_link: mass 0.6852429363 -> 0.120
- link r_hip_twist_link: mass 0.0755193623 -> 0.016
- link r_lower_arm_link: mass 0.3833833954 -> 0.060
- link r_lower_leg_link: mass 0.4326089335 -> 0.080
- link r_shoulder_swing_link: mass 0.0595945816 -> 0.010
- link r_upper_arm_link: mass 0.3822870734 -> 0.070
- link r_upper_leg_link: mass 0.1557654222 -> 0.030
- link torso_link: mass None -> 0.411
